File: KiCad/SignalMixer/SignalMixer.kicad_pcb (KiCad board)
At the start: 2 copper layers, 41 parts, among them J1 Canal 1, J2 Canal 2, J3 Conn_01x02, J4 Saída, SW1 SW_DIP_x08, U1 LM358DT, U2 LM358DT

Commit message: Finalizacao do layout da PCB.
Parts:
- added H1: MountingHole, MountingHole:MountingHole_3.2mm_M3, F.Cu at (129.7, 78.8)
- added H2: MountingHole, MountingHole:MountingHole_3.2mm_M3, F.Cu at (129.7, 126.8)
- added H3: MountingHole, MountingHole:MountingHole_3.2mm_M3, F.Cu at (175.7, 126.8)
- added H4: MountingHole, MountingHole:MountingHole_3.2mm_M3, F.Cu at (175.7, 78.8)
- C1, C2, C3, C4, R1, R10, R11, R12, R13, R14, R15, R16, R17, R18, R19, R2, R20, R21, R22, R23, R24, R3, R4, R5, R6, R7, R8, R9, U1, U2: moved to B.Cu
- moved R10 69.6 mm to (145.9, 110.6), turned to 90 degrees
- moved TP6 68.3 mm to (150.2, 109.8)
- moved J4 65.9 mm to (175.5, 102.6), turned to -90 degrees
- moved R7 58.9 mm to (141.9, 98.6), turned to -90 degrees
- moved R21 54.5 mm to (165.4, 98.6), turned to 90 degrees
- moved J3 52.9 mm to (151.4, 117.1)
- moved R22 52.9 mm to (163.2, 98.6), turned to 90 degrees
- moved R5 52.7 mm to (141.4, 90.6), turned to 90 degrees
- moved TP4 52.0 mm to (150.2, 103.8)
- moved C2 51.7 mm to (161.9, 104.6), turned to 90 degrees
- moved R13 48.0 mm to (145.7, 90.8), turned to -90 degrees
- moved SW1 46.7 mm to (143.7, 93.6), turned to 90 degrees
- moved J2 43.1 mm to (129.6, 113.3), turned to 90 degrees
- moved R14 41.6 mm to (161.9, 90.8), turned to -90 degrees
- moved R24 38.4 mm to (159.2, 110.6), turned to 90 degrees
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Routing:
- net Net-(R14-Pad1): track 0.00 -> 57.6 mm, vias 0 -> 2
- net /SW1_5_P12: track 0.00 -> 54.3 mm, vias 0 -> 1
- net GND: track 0.00 -> 43.9 mm
- net +24V: track 0.00 -> 42.0 mm
- net /SW1_6_P11: track 0.00 -> 38.7 mm, vias 0 -> 3
- net /SW1_2_P15: track 0.00 -> 35.2 mm, vias 0 -> 1
- net /SW1_1_P16: track 0.00 -> 27.0 mm
- net Net-(R11-Pad1): track 0.00 -> 19.5 mm
- net Net-(R20-Pad2): track 0.00 -> 17.8 mm, vias 0 -> 2
- net Net-(J4-Pad1): track 0.00 -> 14.9 mm
- net Net-(C3-Pad2): track 0.00 -> 9.20 mm
- net Net-(R17-Pad2): track 0.00 -> 6.85 mm
- net /SW1_5_P5: track 0.00 -> 4.34 mm
- net /SW1_1_P1: track 0.00 -> 4.34 mm
- net Net-(R10-Pad2): track 0.00 -> 3.15 mm
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- added copper zone on B.Cu, net GNDS
- added copper zone on F.Cu, net GNDS
Other:
- board outline added: 59 x 59 mm
- board text added: "+"
- board text added: "-"
- board text added: "1 2 3 4"
- board text added: "24Vcc"
- board text added: "5 6 7 8"
- board text added: "Eng. Júlio R. R. Santos linkedin.com/in/juliorrsantos"
- board text added: "Misturador de sinais analógicos."
- board text added: "SW1 1 - ON: Canal 1 50Ω| OFF: Canal 1 1MΩ 5 - ON: Canal 2 50Ω| OFF: Canal 2 1MΩ"
- board text added: "SW1 Ganho 2 3 4 Canal 1 6 7 8 Canal 2 ---------------------- OFF OFF OFF {dblquote}infinito{dblquote} (Saturação) ON OFF OFF 1 OFF ON OFF 10 OFF OFF ON 100 ON ON ON 0,9009 ON ON OFF 0,909 ON OFF ON 0,99 OFF ON ON 9,09"
